File: pcb_eagle/OSSC_HDMI_Audio_v1.5_A3a.brd (EAGLE design)
At the start: 29.8 x 24 mm, 29 parts, among them U1 PCM1808, U2 74LVC1G34, U3 MK2507SLF

Commit message: External Masterclock option removed in OSSC firmware v0.75 - PCB files back to A3 - backed up A4 in additional sub-folder
Parts:
- U$1: value OSSC_DIY_AUDIO_OVERLAYDIY-V1.5 -> OSSC_DIY_AUDIO_OVERLAYDIY_V1.5
Connections:
- net N$17: no longer U$1.5
Routing:
- net N$17: track 14.4 -> 10.2 mm
Other:
- board text added: "Rev.: v1.5-A3a"
- board text removed: "Rev.: v1.5-A4a"
Changed lines of the file:
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@@
 <?xml version="1.0" encoding="utf-8"?>
 <!DOCTYPE eagle SYSTEM "eagle.dtd">
-<eagle version="7.6.0">
+<eagle version="7.7.0">
 <drawing>
 <settings>
@@
 </polygon>
 <text x="0.47625" y="7.77875" size="0.8128" layer="25" font="vector" ratio="15">Rev.:
-v1.5-A4a</text>
+v1.5-A3a</text>
 <polygon width="0.1524" layer="41">
 <vertex x="26.51125" y="19.05"/>
@@
 </element>
 <element name="U2" library="OSSC_HDMI_Audio" package="74LVC1G34DCK" value="74LVC1G34" x="7.14375" y="12.065" smashed="yes"/>
-<element name="U$1" library="OSSC_HDMI_Audio" package="OSSC_OVERLAY_V1.5" value="OSSC_DIY_AUDIO_OVERLAYDIY-V1.5" x="22.38375" y="0" smashed="yes"/>
+<element name="U$1" library="OSSC_HDMI_Audio" package="OSSC_OVERLAY_V1.5" value="OSSC_DIY_AUDIO_OVERLAYDIY_V1.5" x="22.38375" y="0" smashed="yes"/>
 </elements>
 <signals>
@@
 <wire x1="22.38375" y1="0" x2="22.38375" y2="3.65125" width="1.076959375" layer="1"/>
 <via x="28.41625" y="12.22375" extent="1-16" drill="0.4572"/>
+<via x="27.305" y="23.495" extent="1-16" drill="0.4572"/>
 <contactref element="U$1" pad="4"/>
-<via x="27.305" y="23.495" extent="1-16" drill="0.4572"/>
 </signal>
 <signal name="N$1">
@@
 <signal name="N$13">
 <contactref element="U1" pad="7"/>
-<contactref element="U$1" pad="10"/>
 <wire x1="22.00875" y1="21.635" x2="20.32" y2="21.635" width="0.254" layer="1"/>
 <via x="20.32" y="21.635" extent="1-16" drill="0.3556"/>
@@
 <wire x1="20.32" y1="21.635" x2="18.7325" y2="21.635" width="0.254" layer="16"/>
 <wire x1="18.18375" y1="22.18375" x2="18.7325" y2="21.635" width="0.254" layer="1"/>
+<contactref element="U$1" pad="10"/>
 </signal>
 <signal name="N$14">
 <contactref element="U1" pad="8"/>
-<contactref element="U$1" pad="11"/>
 <wire x1="16.48375" y1="21.635" x2="17.4175" y2="21.635" width="0.254" layer="1"/>
 <wire x1="17.4175" y1="21.635" x2="18.0975" y2="20.955" width="0.254" layer="1"/>
@@
 <wire x1="19.3675" y1="21.2725" x2="19.3675" y2="23.66625" width="0.254" layer="1"/>
 <wire x1="19.3675" y1="23.66625" x2="19.28375" y2="23.75" width="0.254" layer="1"/>
+<contactref element="U$1" pad="11"/>
 </signal>
 <signal name="N$15">
 <contactref element="U1" pad="9"/>
-<contactref element="U$1" pad="9"/>
 <wire x1="16.48375" y1="20.985" x2="15.5275" y2="20.985" width="0.254" layer="1"/>
 <wire x1="15.5275" y1="20.985" x2="15.24" y2="21.2725" width="0.254" layer="1"/>
@@
 <wire x1="16.66875" y1="22.5425" x2="17.08375" y2="22.9575" width="0.254" layer="1"/>
 <wire x1="17.08375" y1="23.75" x2="17.08375" y2="22.9575" width="0.254" layer="1"/>
+<contactref element="U$1" pad="9"/>
 </signal>
 <signal name="VCC">
@@
 <wire x1="22.00875" y1="20.985" x2="20.19125" y2="20.985" width="0.254" layer="1"/>
 <wire x1="20.19125" y1="20.985" x2="19.05" y2="19.84375" width="0.254" layer="1"/>
-<contactref element="U$1" pad="5"/>
-<wire x1="13.49375" y1="19.84375" x2="13.97" y2="20.32" width="0.254" layer="1"/>
-<wire x1="13.97" y1="20.32" x2="13.97" y2="22.38375" width="0.254" layer="1"/>
-<wire x1="13.97" y1="22.38375" x2="14.76375" y2="23.1775" width="0.254" layer="1"/>
-<wire x1="14.76375" y1="23.1775" x2="14.76375" y2="23.495" width="0.254" layer="1"/>
 </signal>
 <signal name="VCC/2">
